File: Hardware-Project/ADA/Oximeter-Sensor.kicad_sch (KiCad schematic)
At the start: 15 parts

Commit message: Structure Thesis
Model created for the development of my thesis.
Other:
- note added: "Github Version edited..."
- note removed: "Github Version"
Changed lines of the file:
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@@
     (stroke (width 0) (type default) (color 0 0 0 0))
   )
-  (text "Github Version\n" (at 81.28 157.48 0)
+  (text "Github Version\nedited..." (at 81.28 157.48 0)
     (effects (font (size 1.27 1.27)) (justify left bottom))
   )
